File: MX/mx.kicad_pcb (KiCad board)
At the start: 2 copper layers, 315.5 x 155 mm, 190 parts

Commit message: Add files via upload
Parts:
- removed the REF** at (336.2, 121.0)
- removed the REF** at (179.7, 137.0)
- removed the REF** at (272.5, 164.6)
- removed the REF** at (147.3, 116.4)
- removed the REF** at (177.4, 196.9)
- removed the REF** at (163.6, 171.5)
- removed the REF** at (82.6, 119.9)
- removed the REF** at (320.1, 86.4)
- removed the REF** at (171.7, 154.3)
- removed the REF** at (151.2, 125.9)
- removed the REF** at (315.2, 120.9)
- removed the REF** at (344.3, 138.2)
- removed the REF** at (312.9, 161.2)
- removed the REF** at (272.6, 119.7)
- removed the REF** at (107.9, 110.7)
- removed the REF** at (288.8, 109.4)
- removed the REF** at (307.1, 103.6)
- removed the REF** at (304.9, 143.9)
- removed the REF** at (319.6, 112.7)
- removed the REF** at (288.7, 154.2)
- removed the REF** at (112.9, 145.1)
- removed the REF** at (74.6, 137.2)
- removed the REF** at (171.6, 109.4)
- removed the REF** at (264.4, 147.3)
- removed the REF** at (129.0, 110.6)
- removed the REF** at (361.5, 130.2)
- removed the REF** at (139.3, 133.6)
- removed the REF** at (134.9, 115.6)
- removed the REF** at (353.5, 112.9)
- removed the REF** at (299.1, 86.3)
- removed the REF** at (98.7, 85.4)
- removed the REF** at (296.8, 126.7)
- removed the REF** at (121.0, 127.9)
- removed the REF** at (280.7, 92.1)
- removed the REF** at (248.3, 112.8)
- removed the REF** at (137.1, 93.3)
- removed the REF** at (155.5, 144.0)
- removed the REF** at (257.3, 206.4)
- removed the REF** at (131.2, 150.9)
- removed the REF** at (90.7, 102.7)
- removed the REF** at (91.8, 145.2)
- removed the REF** at (280.6, 137.0)
- removed the REF** at (345.4, 95.7)
- removed the REF** at (167.4, 136.2)
- removed the REF** at (336.9, 104.6)
- removed the REF** at (154.1, 193.8)
- removed the REF** at (163.5, 126.7)
- removed the REF** at (323.2, 138.1)
- removed the REF** at (116.0, 93.4)
- removed the REF** at (99.9, 128.0)
- removed the REF** at (264.5, 102.4)
- removed the REF** at (331.3, 155.4)
- removed the REF** at (123.2, 168.2)
- removed the REF** at (147.4, 161.2)
- removed the REF** at (187.8, 119.8)
- removed the REF** at (298.6, 112.6)
- removed the REF** at (296.7, 171.5)
- removed the REF** at (256.4, 130.0)
- removed the REF** at (328.2, 103.7)
- removed the REF** at (155.4, 99.1)
- removed the REF** at (278.1, 181.5)
- removed the REF** at (337.4, 78.4)
- removed the REF** at (104.9, 162.4)
- removed the REF** at (139.4, 178.5)
- added G***: LOGO, Library:mankini_logo, F.Cu at (207.7, 194.7)
- added REF**: VIA-0.6mm, ceoloide:VIA-0.6mm, F.Cu at (239.4, 147.1)
- added REF**: VIA-0.6mm, ceoloide:VIA-0.6mm, F.Cu at (173.9, 151.6)
- added REF**: VIA-0.6mm, VIA-0.6mm, F.Cu at (152.5, 107.3)
- added REF**: VIA-0.6mm, VIA-0.6mm, F.Cu at (174.6, 205.1)
- added REF**: VIA-0.6mm, ceoloide:VIA-0.6mm, F.Cu at (254.6, 179.7)
- added REF**: VIA-0.6mm, VIA-0.6mm, F.Cu at (110.1, 153.3)
- added REF**: VIA-0.6mm, ceoloide:VIA-0.6mm, F.Cu at (246.6, 162.5)
- added REF**: VIA-0.6mm, VIA-0.6mm, F.Cu at (285.8, 162.4)
- added REF**: VIA-0.6mm, VIA-0.6mm, F.Cu at (292.3, 122.4)
- added REF**: VIA-0.6mm, ceoloide:VIA-0.6mm, F.Cu at (241.5, 151.6)
- added REF**: VIA-0.6mm, VIA-0.6mm, F.Cu at (245.5, 120.9)
- added REF**: VIA-0.6mm, VIA-0.6mm, F.Cu at (341.4, 146.4)
- added REF**: VIA-0.6mm, VIA-0.6mm, F.Cu at (160.7, 134.9)
- added REF**: VIA-0.6mm, VIA-0.6mm, F.Cu at (136.5, 186.7)
- added REF**: VIA-0.6mm, ceoloide:VIA-0.6mm, F.Cu at (176.0, 147.1)
- added REF**: VIA-0.6mm, VIA-0.6mm, F.Cu at (313.3, 122.5)
- added REF**: VIA-0.6mm, VIA-0.6mm, F.Cu at (143.8, 134.8)
- added REF**: VIA-0.6mm, VIA-0.6mm, F.Cu at (79.8, 128.1)
- added REF**: VIA-0.6mm, VIA-0.6mm, F.Cu at (312.3, 129.1)
- added REF**: VIA-0.6mm, VIA-0.6mm, F.Cu at (342.6, 103.8)
- added REF**: VIA-0.6mm, VIA-0.6mm, F.Cu at (144.5, 124.6)
- added REF**: VIA-0.6mm, VIA-0.6mm, F.Cu at (254.4, 214.6)
- added REF**: VIA-0.6mm, VIA-0.6mm, F.Cu at (317.3, 94.6)
- added REF**: VIA-0.6mm, VIA-0.6mm, F.Cu at (286.0, 117.6)
- added REF**: VIA-0.6mm, VIA-0.6mm, F.Cu at (277.9, 100.3)
- added REF**: VIA-0.6mm, VIA-0.6mm, F.Cu at (126.2, 118.8)
- added REF**: VIA-0.6mm, VIA-0.6mm, F.Cu at (269.7, 127.9)
- added REF**: VIA-0.6mm, VIA-0.6mm, F.Cu at (333.4, 129.2)
- added REF**: VIA-0.6mm, VIA-0.6mm, F.Cu at (144.6, 169.4)
- added REF**: VIA-0.6mm, VIA-0.6mm, F.Cu at (120.3, 176.4)
- added REF**: VIA-0.6mm, VIA-0.6mm, F.Cu at (185.0, 127.9)
- added REF**: VIA-0.6mm, VIA-0.6mm, F.Cu at (330.6, 114.4)
- added REF**: VIA-0.6mm, VIA-0.6mm, F.Cu at (294.0, 134.8)
- added REF**: VIA-0.6mm, VIA-0.6mm, F.Cu at (97.0, 136.2)
- added REF**: VIA-0.6mm, VIA-0.6mm, F.Cu at (176.9, 145.2)
- added REF**: VIA-0.6mm, ceoloide:VIA-0.6mm, F.Cu at (230.5, 127.9)
- added REF**: VIA-0.6mm, VIA-0.6mm, F.Cu at (105.1, 118.9)
- added REF**: VIA-0.6mm, VIA-0.6mm, F.Cu at (275.2, 189.7)
- added REF**: VIA-0.6mm, VIA-0.6mm, F.Cu at (113.1, 101.6)
- added REF**: VIA-0.6mm, VIA-0.6mm, F.Cu at (261.7, 110.6)
- added REF**: VIA-0.6mm, VIA-0.6mm, F.Cu at (325.3, 111.9)
- added REF**: VIA-0.6mm, ceoloide:VIA-0.6mm, F.Cu at (240.5, 149.3)
- added REF**: VIA-0.6mm, VIA-0.6mm, F.Cu at (320.4, 146.3)
- added REF**: VIA-0.6mm, VIA-0.6mm, F.Cu at (118.1, 136.0)
- added REF**: VIA-0.6mm, VIA-0.6mm, F.Cu at (328.4, 163.6)
- added REF**: VIA-0.6mm, VIA-0.6mm, F.Cu at (168.7, 117.6)
- added REF**: VIA-0.6mm, VIA-0.6mm, F.Cu at (89.0, 153.4)
- added REF**: VIA-0.6mm, VIA-0.6mm, F.Cu at (277.8, 145.2)
- added REF**: VIA-0.6mm, VIA-0.6mm, F.Cu at (296.2, 94.5)
- added REF**: VIA-0.6mm, VIA-0.6mm, F.Cu at (261.6, 155.5)
- added REF**: VIA-0.6mm, VIA-0.6mm, F.Cu at (253.5, 138.2)
- added REF**: VIA-0.6mm, VIA-0.6mm, F.Cu at (87.8, 110.8)
- added REF**: VIA-0.6mm, VIA-0.6mm, F.Cu at (102.0, 170.6)
- added REF**: VIA-0.6mm, VIA-0.6mm, F.Cu at (128.4, 159.1)
- added REF**: VIA-0.6mm, VIA-0.6mm, F.Cu at (152.6, 152.2)
- added REF**: VIA-0.6mm, VIA-0.6mm, F.Cu at (302.1, 152.1)
- added REF**: VIA-0.6mm, VIA-0.6mm, F.Cu at (127.6, 124.5)
- added REF**: VIA-0.6mm, VIA-0.6mm, F.Cu at (168.9, 162.5)
- added REF**: VIA-0.6mm, VIA-0.6mm, F.Cu at (304.3, 111.8)
- added REF**: VIA-0.6mm, VIA-0.6mm, F.Cu at (160.8, 179.7)
- added REF**: VIA-0.6mm, ceoloide:VIA-0.6mm, F.Cu at (175.0, 149.3)
- added REF**: VIA-0.6mm, VIA-0.6mm, F.Cu at (134.2, 101.5)
- added REF**: VIA-0.6mm, VIA-0.6mm, F.Cu at (350.7, 121.1)
- added REF**: VIA-0.6mm, ceoloide:VIA-0.6mm, F.Cu at (238.5, 145.2)
- added REF**: VIA-0.6mm, VIA-0.6mm, F.Cu at (310.1, 169.4)
- added REF**: VIA-0.6mm, VIA-0.6mm, F.Cu at (160.0, 145.1)
- added REF**: VIA-0.6mm, VIA-0.6mm, F.Cu at (136.4, 141.8)
- added REF**: VIA-0.6mm, VIA-0.6mm, F.Cu at (334.6, 86.6)
- added REF**: VIA-0.6mm, VIA-0.6mm, F.Cu at (95.9, 93.6)
- added REF**: VIA-0.6mm, VIA-0.6mm, F.Cu at (358.7, 138.4)
- added REF**: VIA-0.6mm, VIA-0.6mm, F.Cu at (71.7, 145.4)
- added REF**: VIA-0.6mm, VIA-0.6mm, F.Cu at (293.9, 179.7)
- added REF**: VIA-0.6mm, VIA-0.6mm, F.Cu at (269.6, 172.7)
- added REF**: VIA-0.6mm, VIA-0.6mm, F.Cu at (151.3, 202.0)
- S1, S10, S11, S12, S13, S14, S15, S16, S17, S18, S19, S2, S20, S21, S22, S23, S24, S25, S26, S27, S28, S29, S3, S30, S31, S32, S33, S34, S35, S36, S37, S38, S39, S4, S40, S41, S42, S43, S44, S45, S46, S47, S48, S49, S5, S50, S51, S52, S53, S54, S55, S56, S57, S58, S6, S7, S8, S9: footprint ceoloide:switch_choc_v1_v2 -> ceoloide:switch_mx
- moved D32 8.66 mm to (341.1, 100.7)
- moved D34 8.66 mm to (340.0, 143.3)
- moved S12 8.66 mm to (120.4, 111.7)
- moved _70 8.66 mm to (336.9, 133.6)
- moved S21 8.66 mm to (146.8, 145.0)
- moved S5 8.66 mm to (83.2, 146.3)
- moved S38 8.66 mm to (319.2, 163.5)
- moved S46 8.66 mm to (276.8, 117.4)
- moved S22 8.66 mm to (154.9, 127.8)
- moved D4 8.66 mm to (97.4, 90.4)
- moved S11 8.66 mm to (112.3, 128.9)
- moved D22 8.66 mm to (162.2, 131.7)
- moved S29 8.66 mm to (165.5, 206.6)
- moved S32 8.66 mm to (333.4, 103.7)
- moved S9 8.66 mm to (96.2, 163.5)
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Routing:
- net G6: track 604.8 -> 533.3 mm
- net G5: track 648.7 -> 583.2 mm
- net G27: track 551.2 -> 510.1 mm
- net G4: track 660.8 -> 633.6 mm
- net G26: track 472.8 -> 457.8 mm
- net G18: track 399.3 -> 412.0 mm
- net G9: track 187.1 -> 183.4 mm
- net G2: track 191.9 -> 195.6 mm
- net index_num: track 2.60 -> 6.17 mm
- net ring_home: track 2.60 -> 6.16 mm
- net outer_top: track 2.60 -> 6.15 mm
- net G28: track 157.7 -> 161.3 mm
- net mirror_inner_top: track 2.60 -> 6.13 mm
- net ring_top: track 2.60 -> 6.13 mm
- net index_top: track 2.60 -> 6.13 mm
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Other:
- board text added: "Cherry MX version"
- board text added: "THE MANKINI"
- board text added: "by @jaybuilds"
- board text added: "https://github.com/jaybuilds222/Mankini"
- board text removed: "THE MANKINI - MX"
- board text removed: "by @Jaybuilds"
- board text removed: "https:/github.com/jaybuildsstuff/Mankini/MX"
- board text removed: "info@jaybuilds.com"

Commit message: Add files via upload
Parts:
- removed G***: LOGO, Library:mankini_logo
- removed the REF** at (239.4, 147.1)
- removed the REF** at (173.9, 151.6)
- removed the REF** at (152.5, 107.3)
- removed the REF** at (174.6, 205.1)
- removed the REF** at (254.6, 179.7)
- removed the REF** at (110.1, 153.3)
- removed the REF** at (246.6, 162.5)
- removed the REF** at (285.8, 162.4)
- removed the REF** at (292.3, 122.4)
- removed the REF** at (241.5, 151.6)
- removed the REF** at (245.5, 120.9)
- removed the REF** at (341.4, 146.4)
- removed the REF** at (160.7, 134.9)
- removed the REF** at (136.5, 186.7)
- removed the REF** at (176.0, 147.1)
- removed the REF** at (313.3, 122.5)
- removed the REF** at (143.8, 134.8)
- removed the REF** at (79.8, 128.1)
- removed the REF** at (312.3, 129.1)
- removed the REF** at (342.6, 103.8)
- removed the REF** at (144.5, 124.6)
- removed the REF** at (254.4, 214.6)
- removed the REF** at (317.3, 94.6)
- removed the REF** at (286.0, 117.6)
- removed the REF** at (277.9, 100.3)
- removed the REF** at (126.2, 118.8)
- removed the REF** at (269.7, 127.9)
- removed the REF** at (333.4, 129.2)
- removed the REF** at (144.6, 169.4)
- removed the REF** at (120.3, 176.4)
- removed the REF** at (185.0, 127.9)
- removed the REF** at (330.6, 114.4)
- removed the REF** at (294.0, 134.8)
- removed the REF** at (97.0, 136.2)
- removed the REF** at (176.9, 145.2)
- removed the REF** at (230.5, 127.9)
- removed the REF** at (105.1, 118.9)
- removed the REF** at (275.2, 189.7)
- removed the REF** at (113.1, 101.6)
- removed the REF** at (261.7, 110.6)
- removed the REF** at (325.3, 111.9)
- removed the REF** at (240.5, 149.3)
- removed the REF** at (320.4, 146.3)
- removed the REF** at (118.1, 136.0)
- removed the REF** at (328.4, 163.6)
- removed the REF** at (168.7, 117.6)
- removed the REF** at (89.0, 153.4)
- removed the REF** at (277.8, 145.2)
- removed the REF** at (296.2, 94.5)
- removed the REF** at (261.6, 155.5)
- removed the REF** at (253.5, 138.2)
- removed the REF** at (87.8, 110.8)
- removed the REF** at (102.0, 170.6)
- removed the REF** at (128.4, 159.1)
- removed the REF** at (152.6, 152.2)
- removed the REF** at (302.1, 152.1)
- removed the REF** at (127.6, 124.5)
- removed the REF** at (168.9, 162.5)
- removed the REF** at (304.3, 111.8)
- removed the REF** at (160.8, 179.7)
- removed the REF** at (175.0, 149.3)
- removed the REF** at (134.2, 101.5)
- removed the REF** at (350.7, 121.1)
- removed the REF** at (238.5, 145.2)
- removed the REF** at (310.1, 169.4)
- removed the REF** at (160.0, 145.1)
- removed the REF** at (136.4, 141.8)
- removed the REF** at (334.6, 86.6)
- removed the REF** at (95.9, 93.6)
- removed the REF** at (358.7, 138.4)
- removed the REF** at (71.7, 145.4)
- removed the REF** at (293.9, 179.7)
- removed the REF** at (269.6, 172.7)
- removed the REF** at (151.3, 202.0)
- added REF**: VIA-0.6mm, VIA-0.6mm, F.Cu at (114.6, 154.6)
- added REF**: VIA-0.6mm, VIA-0.6mm, F.Cu at (173.4, 163.7)
- added REF**: VIA-0.6mm, VIA-0.6mm, F.Cu at (347.2, 105.1)
- added REF**: VIA-0.6mm, VIA-0.6mm, F.Cu at (316.9, 130.3)
- added REF**: VIA-0.6mm, VIA-0.6mm, F.Cu at (336.0, 118.1)
- added REF**: VIA-0.6mm, VIA-0.6mm, F.Cu at (155.8, 203.3)
- added REF**: VIA-0.6mm, VIA-0.6mm, F.Cu at (84.3, 129.4)
- added REF**: VIA-0.6mm, VIA-0.6mm, F.Cu at (141.0, 143.1)
- added REF**: VIA-0.6mm, VIA-0.6mm, F.Cu at (92.4, 112.1)
- added REF**: VIA-0.6mm, VIA-0.6mm, F.Cu at (279.8, 191.0)
- added REF**: VIA-0.6mm, VIA-0.6mm, F.Cu at (282.4, 146.4)
- added REF**: VIA-0.6mm, VIA-0.6mm, F.Cu at (290.5, 118.8)
- added REF**: VIA-0.6mm, VIA-0.6mm, F.Cu at (338.0, 130.4)
- added REF**: VIA-0.6mm, VIA-0.6mm, F.Cu at (164.3, 146.2)
- added REF**: VIA-0.6mm, VIA-0.6mm, F.Cu at (321.9, 95.9)
- added REF**: VIA-0.6mm, VIA-0.6mm, F.Cu at (117.7, 102.9)
- added REF**: VIA-0.6mm, VIA-0.6mm, F.Cu at (141.1, 187.9)
- added REF**: VIA-0.6mm, VIA-0.6mm, F.Cu at (339.1, 87.8)
- added REF**: VIA-0.6mm, VIA-0.6mm, F.Cu at (314.7, 170.6)
- added REF**: VIA-0.6mm, VIA-0.6mm, F.Cu at (133.0, 160.3)
- added REF**: VIA-0.6mm, VIA-0.6mm, F.Cu at (149.1, 125.8)
- added REF**: VIA-0.6mm, VIA-0.6mm, F.Cu at (308.8, 113.0)
- added REF**: VIA-0.6mm, VIA-0.6mm, F.Cu at (274.2, 174.0)
- added REF**: VIA-0.6mm, VIA-0.6mm, F.Cu at (333.0, 164.8)
- added REF**: VIA-0.6mm, VIA-0.6mm, F.Cu at (181.5, 146.5)
- added REF**: VIA-0.6mm, VIA-0.6mm, F.Cu at (250.1, 122.2)
- added REF**: VIA-0.6mm, VIA-0.6mm, F.Cu at (130.7, 120.0)
- added REF**: VIA-0.6mm, VIA-0.6mm, F.Cu at (157.1, 108.6)
- added REF**: VIA-0.6mm, VIA-0.6mm, F.Cu at (298.6, 136.1)
- added REF**: VIA-0.6mm, VIA-0.6mm, F.Cu at (100.4, 94.8)
- added REF**: VIA-0.6mm, VIA-0.6mm, F.Cu at (355.2, 122.4)
- added REF**: VIA-0.6mm, VIA-0.6mm, F.Cu at (148.1, 135.9)
- added REF**: VIA-0.6mm, VIA-0.6mm, F.Cu at (258.1, 139.5)
- added REF**: VIA-0.6mm, VIA-0.6mm, F.Cu at (363.3, 139.6)
- added REF**: VIA-0.6mm, VIA-0.6mm, F.Cu at (324.9, 147.6)
- added REF**: VIA-0.6mm, VIA-0.6mm, F.Cu at (300.8, 95.8)
- added REF**: VIA-0.6mm, VIA-0.6mm, F.Cu at (165.3, 136.1)
- added REF**: VIA-0.6mm, VIA-0.6mm, F.Cu at (122.7, 137.3)
- added REF**: VIA-0.6mm, VIA-0.6mm, F.Cu at (318.7, 126.1)
- added REF**: VIA-0.6mm, VIA-0.6mm, F.Cu at (109.7, 120.1)
- added REF**: VIA-0.6mm, VIA-0.6mm, F.Cu at (124.9, 177.6)
- added REF**: VIA-0.6mm, VIA-0.6mm, F.Cu at (106.6, 171.8)
- added REF**: VIA-0.6mm, VIA-0.6mm, F.Cu at (282.5, 101.6)
- added REF**: VIA-0.6mm, VIA-0.6mm, F.Cu at (101.6, 137.4)
- added REF**: VIA-0.6mm, VIA-0.6mm, F.Cu at (157.2, 153.4)
- added REF**: VIA-0.6mm, VIA-0.6mm, F.Cu at (298.5, 180.9)
- added REF**: VIA-0.6mm, VIA-0.6mm, F.Cu at (189.5, 129.2)
- added REF**: VIA-0.6mm, VIA-0.6mm, F.Cu at (290.4, 163.7)
- added REF**: VIA-0.6mm, VIA-0.6mm, F.Cu at (138.8, 102.8)
- added REF**: VIA-0.6mm, VIA-0.6mm, F.Cu at (149.2, 170.7)
- added REF**: VIA-0.6mm, VIA-0.6mm, F.Cu at (306.6, 153.4)
- added REF**: VIA-0.6mm, VIA-0.6mm, F.Cu at (266.2, 156.7)
- added REF**: VIA-0.6mm, VIA-0.6mm, F.Cu at (259.0, 215.9)
- added REF**: VIA-0.6mm, VIA-0.6mm, F.Cu at (329.9, 113.1)
- added REF**: VIA-0.6mm, VIA-0.6mm, F.Cu at (266.3, 111.9)
- added REF**: VIA-0.6mm, VIA-0.6mm, F.Cu at (93.6, 154.7)
- added REF**: VIA-0.6mm, VIA-0.6mm, F.Cu at (76.3, 146.6)
- added REF**: VIA-0.6mm, VIA-0.6mm, F.Cu at (165.4, 181.0)
- added REF**: VIA-0.6mm, VIA-0.6mm, F.Cu at (173.3, 118.9)
- added REF**: VIA-0.6mm, VIA-0.6mm, F.Cu at (346.0, 147.7)
- added REF**: VIA-0.6mm, VIA-0.6mm, F.Cu at (179.1, 206.4)
- added REF**: VIA-0.6mm, VIA-0.6mm, F.Cu at (274.3, 129.1)
- added REF**: VIA-0.6mm, VIA-0.6mm, F.Cu at (297.7, 126.0)
- added REF**: VIA-0.6mm, VIA-0.6mm, F.Cu at (131.9, 125.6)
- D1, D10, D11, D12, D13, D14, D15, D16, D17, D18, D19, D2, D20, D21, D22, D23, D24, D25, D26, D27, D28, D29, D3, D30, D31, D32, D33, D34, D35, D36, D37, D38, D39, D4, D40, D41, D42, D43, D44, D45, D46, D47, D48, D49, D5, D50, D51, D52, D53, D54, D55, D56, D57, D58, D6, D7, D8, D9: footprint ceoloide:diode_tht_sod123 -> jaybuilds:diode_tht_sod123
- MCU1: footprint ceoloide:mcu_nice_nano -> jaybuilds:mcu_rp2040
- RST1: footprint ceoloide:reset_switch_tht_top -> jaybuilds:reset_switch_tht_top
- S1, S10, S11, S12, S13, S14, S15, S16, S17, S18, S19, S2, S20, S21, S22, S23, S24, S25, S26, S27, S28, S29, S3, S30, S31, S32, S33, S34, S35, S36, S37, S38, S39, S4, S40, S41, S42, S43, S44, S45, S46, S47, S48, S49, S5, S50, S51, S52, S53, S54, S55, S56, S57, S58, S6, S7, S8, S9: footprint ceoloide:switch_mx -> jaybuilds:switch_mx
- moved S46 4.74 mm to (281.3, 118.7)
- moved D56 4.74 mm to (248.6, 119.0)
- moved D27 4.74 mm to (191.0, 126.0)
- moved D53 4.74 mm to (272.7, 170.8)
- moved D13 4.74 mm to (140.3, 99.6)
- moved S38 4.74 mm to (323.8, 164.7)
- moved D36 4.74 mm to (328.4, 110.0)
- moved S20 4.74 mm to (143.4, 163.5)
- moved S13 4.74 mm to (133.0, 95.6)
- moved D41 4.74 mm to (307.4, 109.9)
- moved D7 4.74 mm to (111.1, 117.0)
- moved D9 4.74 mm to (108.1, 168.7)
- moved S58 4.74 mm to (254.5, 207.8)
- moved S41 4.74 mm to (299.7, 112.9)
- moved D4 4.74 mm to (101.9, 91.7)
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Routing:
- net G4: track 633.6 -> 0.00 mm
- net G5: track 583.2 -> 0.00 mm
- net G6: track 533.3 -> 0.00 mm
- net G27: track 510.1 -> 0.00 mm
- net G26: track 457.8 -> 0.00 mm
- net G18: track 412.0 -> 0.00 mm
- net G2: track 195.6 -> 0.00 mm
- net G8: track 188.3 -> 0.00 mm
- net G9: track 183.4 -> 0.00 mm
- net G29: track 180.0 -> 0.00 mm
- net G3: track 176.1 -> 0.00 mm
- net G19: track 171.8 -> 0.00 mm
- net G7: track 168.6 -> 0.00 mm
- net G10: track 165.4 -> 0.00 mm
- net G28: track 161.3 -> 0.00 mm
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Other:
- rule pad_to_mask_clearance: 0 -> 0.05
- board text removed: "Cherry MX version"
- board text removed: "JLCJLCJLCJLC"
- board text removed: "THE MANKINI"
- board text removed: "by @jaybuilds"
- board text removed: "https://github.com/jaybuilds222/Mankini"

Commit message: Add files via upload
Parts:
- removed the REF** at (114.6, 154.6)
- removed the REF** at (173.4, 163.7)
- removed the REF** at (347.2, 105.1)
- removed the REF** at (316.9, 130.3)
- removed the REF** at (336.0, 118.1)
- removed the REF** at (155.8, 203.3)
- removed the REF** at (84.3, 129.4)
- removed the REF** at (141.0, 143.1)
- removed the REF** at (92.4, 112.1)
- removed the REF** at (279.8, 191.0)
- removed the REF** at (282.4, 146.4)
- removed the REF** at (290.5, 118.8)
- removed the REF** at (338.0, 130.4)
- removed the REF** at (164.3, 146.2)
- removed the REF** at (321.9, 95.9)
- removed the REF** at (117.7, 102.9)
- removed the REF** at (141.1, 187.9)
- removed the REF** at (339.1, 87.8)
- removed the REF** at (314.7, 170.6)
- removed the REF** at (133.0, 160.3)
- removed the REF** at (149.1, 125.8)
- removed the REF** at (308.8, 113.0)
- removed the REF** at (274.2, 174.0)
- removed the REF** at (333.0, 164.8)
- removed the REF** at (181.5, 146.5)
- removed the REF** at (250.1, 122.2)
- removed the REF** at (130.7, 120.0)
- removed the REF** at (157.1, 108.6)
- removed the REF** at (298.6, 136.1)
- removed the REF** at (100.4, 94.8)
- removed the REF** at (355.2, 122.4)
- removed the REF** at (148.1, 135.9)
- removed the REF** at (258.1, 139.5)
- removed the REF** at (363.3, 139.6)
- removed the REF** at (324.9, 147.6)
- removed the REF** at (300.8, 95.8)
- removed the REF** at (165.3, 136.1)
- removed the REF** at (122.7, 137.3)
- removed the REF** at (318.7, 126.1)
- removed the REF** at (109.7, 120.1)
- removed the REF** at (124.9, 177.6)
- removed the REF** at (106.6, 171.8)
- removed the REF** at (282.5, 101.6)
- removed the REF** at (101.6, 137.4)
- removed the REF** at (157.2, 153.4)
- removed the REF** at (298.5, 180.9)
- removed the REF** at (189.5, 129.2)
- removed the REF** at (290.4, 163.7)
- removed the REF** at (138.8, 102.8)
- removed the REF** at (149.2, 170.7)
- removed the REF** at (306.6, 153.4)
- removed the REF** at (266.2, 156.7)
- removed the REF** at (259.0, 215.9)
- removed the REF** at (329.9, 113.1)
- removed the REF** at (266.3, 111.9)
- removed the REF** at (93.6, 154.7)
- removed the REF** at (76.3, 146.6)
- removed the REF** at (165.4, 181.0)
- removed the REF** at (173.3, 118.9)
- removed the REF** at (346.0, 147.7)
- removed the REF** at (179.1, 206.4)
- removed the REF** at (274.3, 129.1)
- removed the REF** at (297.7, 126.0)
- removed the REF** at (131.9, 125.6)
- added REF**: VIA-0.6mm, VIA-0.6mm, F.Cu at (186.7, 125.3)
- added REF**: VIA-0.6mm, VIA-0.6mm, F.Cu at (255.3, 135.6)
- added REF**: VIA-0.6mm, VIA-0.6mm, F.Cu at (335.1, 126.5)
- added REF**: VIA-0.6mm, VIA-0.6mm, F.Cu at (360.5, 135.7)
- added REF**: VIA-0.6mm, VIA-0.6mm, F.Cu at (138.2, 139.2)
- added REF**: VIA-0.6mm, VIA-0.6mm, F.Cu at (247.2, 118.3)
- added REF**: VIA-0.6mm, VIA-0.6mm, F.Cu at (154.3, 104.7)
- added REF**: VIA-0.6mm, VIA-0.6mm, F.Cu at (295.8, 132.2)
- added REF**: VIA-0.6mm, VIA-0.6mm, F.Cu at (90.7, 150.8)
- added REF**: VIA-0.6mm, VIA-0.6mm, F.Cu at (322.1, 143.7)
- added REF**: VIA-0.6mm, VIA-0.6mm, F.Cu at (295.7, 177.1)
- added REF**: VIA-0.6mm, VIA-0.6mm, F.Cu at (294.8, 122.2)
- added REF**: VIA-0.6mm, VIA-0.6mm, F.Cu at (146.2, 121.9)
- added REF**: VIA-0.6mm, VIA-0.6mm, F.Cu at (256.2, 212.0)
- added REF**: VIA-0.6mm, VIA-0.6mm, F.Cu at (271.4, 170.1)
- added REF**: VIA-0.6mm, VIA-0.6mm, F.Cu at (343.2, 143.8)
- added REF**: VIA-0.6mm, VIA-0.6mm, F.Cu at (279.5, 142.5)
- added REF**: VIA-0.6mm, VIA-0.6mm, F.Cu at (89.6, 108.2)
- added REF**: VIA-0.6mm, VIA-0.6mm, F.Cu at (178.7, 142.6)
- added REF**: VIA-0.6mm, VIA-0.6mm, F.Cu at (98.8, 133.5)
- added REF**: VIA-0.6mm, VIA-0.6mm, F.Cu at (271.5, 125.3)
- added REF**: VIA-0.6mm, VIA-0.6mm, F.Cu at (122.1, 173.7)
- added REF**: VIA-0.6mm, VIA-0.6mm, F.Cu at (306.0, 109.2)
- added REF**: VIA-0.6mm, VIA-0.6mm, F.Cu at (154.4, 149.5)
- added REF**: VIA-0.6mm, VIA-0.6mm, F.Cu at (81.5, 125.5)
- added REF**: VIA-0.6mm, VIA-0.6mm, F.Cu at (263.3, 152.8)
- added REF**: VIA-0.6mm, VIA-0.6mm, F.Cu at (311.9, 166.7)
- added REF**: VIA-0.6mm, VIA-0.6mm, F.Cu at (146.3, 166.8)
- added REF**: VIA-0.6mm, VIA-0.6mm, F.Cu at (170.5, 115.0)
- added REF**: VIA-0.6mm, VIA-0.6mm, F.Cu at (315.9, 122.3)
- added REF**: VIA-0.6mm, VIA-0.6mm, F.Cu at (298.0, 91.9)
- added REF**: VIA-0.6mm, VIA-0.6mm, F.Cu at (145.3, 132.0)
- added REF**: VIA-0.6mm, VIA-0.6mm, F.Cu at (73.5, 142.7)
- added REF**: VIA-0.6mm, VIA-0.6mm, F.Cu at (352.4, 118.5)
- added REF**: VIA-0.6mm, VIA-0.6mm, F.Cu at (279.7, 97.7)
- added REF**: VIA-0.6mm, VIA-0.6mm, F.Cu at (319.0, 92.0)
- added REF**: VIA-0.6mm, VIA-0.6mm, F.Cu at (106.8, 116.3)
- added REF**: VIA-0.6mm, VIA-0.6mm, F.Cu at (277.0, 187.1)
- added REF**: VIA-0.6mm, VIA-0.6mm, F.Cu at (130.1, 156.5)
- added REF**: VIA-0.6mm, VIA-0.6mm, F.Cu at (162.6, 177.1)
- added REF**: VIA-0.6mm, VIA-0.6mm, F.Cu at (176.3, 202.5)
- added REF**: VIA-0.6mm, VIA-0.6mm, F.Cu at (138.3, 184.0)
- added REF**: VIA-0.6mm, VIA-0.6mm, F.Cu at (344.4, 101.2)
- added REF**: VIA-0.6mm, VIA-0.6mm, F.Cu at (314.1, 126.4)
- added REF**: VIA-0.6mm, VIA-0.6mm, F.Cu at (111.8, 150.7)
- added REF**: VIA-0.6mm, VIA-0.6mm, F.Cu at (103.8, 167.9)
- added REF**: VIA-0.6mm, VIA-0.6mm, F.Cu at (327.1, 109.3)
- added REF**: traces, Library:traces, F.Cu at (209.5, 207.0)
- added REF**: VIA-0.6mm, VIA-0.6mm, F.Cu at (170.6, 159.8)
- added REF**: VIA-0.6mm, VIA-0.6mm, F.Cu at (303.8, 149.5)
- added REF**: VIA-0.6mm, VIA-0.6mm, F.Cu at (287.6, 159.8)
- added REF**: VIA-0.6mm, VIA-0.6mm, F.Cu at (287.7, 114.9)
- added REF**: VIA-0.6mm, VIA-0.6mm, F.Cu at (114.9, 99.0)
- added REF**: VIA-0.6mm, VIA-0.6mm, F.Cu at (97.6, 90.9)
- added REF**: VIA-0.6mm, VIA-0.6mm, F.Cu at (263.4, 108.0)
- added REF**: VIA-0.6mm, VIA-0.6mm, F.Cu at (119.9, 133.4)
- added REF**: VIA-0.6mm, VIA-0.6mm, F.Cu at (333.2, 114.2)
- added REF**: VIA-0.6mm, VIA-0.6mm, F.Cu at (129.1, 121.7)
- added REF**: VIA-0.6mm, VIA-0.6mm, F.Cu at (127.9, 116.2)
- added REF**: VIA-0.6mm, VIA-0.6mm, F.Cu at (153.0, 199.4)
- added REF**: VIA-0.6mm, VIA-0.6mm, F.Cu at (136.0, 98.9)
- added REF**: VIA-0.6mm, VIA-0.6mm, F.Cu at (336.3, 83.9)
- added REF**: VIA-0.6mm, VIA-0.6mm, F.Cu at (161.5, 142.4)
- added REF**: VIA-0.6mm, VIA-0.6mm, F.Cu at (330.2, 161.0)
- added REF**: VIA-0.6mm, VIA-0.6mm, F.Cu at (162.4, 132.3)
- moved D21 4.79 mm to (155.9, 146.3)
- moved D25 4.79 mm to (172.1, 156.7)
- moved D30 4.79 mm to (359.0, 132.6)
- moved D31 4.79 mm to (350.9, 115.3)
- moved D39 4.79 mm to (320.7, 140.5)
- moved D40 4.79 mm to (312.6, 123.3)
- moved D41 4.79 mm to (304.5, 106.0)
- moved D44 4.79 mm to (302.3, 146.3)
- moved D45 4.79 mm to (294.3, 129.0)
- moved D49 4.79 mm to (286.1, 156.6)
- moved D50 4.79 mm to (278.1, 139.4)
- moved D56 4.79 mm to (245.8, 115.1)
- moved S21 4.79 mm to (148.6, 142.4)
- moved S30 4.79 mm to (351.3, 135.6)
- moved S39 4.79 mm to (312.9, 143.6)
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